Commit message: Add Gazebo implementation branch updates

File: src/quadruped_ros2_control-humble/descriptions/unitree/go1_description/urdf/robot.urdf (robot description, URDF)
Before this commit: robot go1, 46 links, 45 joints
Links:
- link FL_calf: geometry visual mesh filename=file:///home/tlab-uav/ros2_ws/install/go1_description/share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 scale=1 1 1
- link FL_thigh: geometry visual mesh filename=file:///home/tlab-uav/ros2_ws/install/go1_description/share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 scale=1 1 1
- link FR_calf: geometry visual mesh filename=file:///home/tlab-uav/ros2_ws/install/go1_description/share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 scale=1 1 1
- link FR_thigh: geometry visual mesh filename=file:///home/tlab-uav/ros2_ws/install/go1_description/share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 scale=1 1 1
- link RL_calf: geometry visual mesh filename=file:///home/tlab-uav/ros2_ws/install/go1_description/share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 scale=1 1 1
- link RL_thigh: geometry visual mesh filename=file:///home/tlab-uav/ros2_ws/install/go1_description/share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 scale=1 1 1
- link RR_calf: geometry visual mesh filename=file:///home/tlab-uav/ros2_ws/install/go1_description/share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 scale=1 1 1
- link RR_thigh: geometry visual mesh filename=file:///home/tlab-uav/ros2_ws/install/go1_description/share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 scale=1 1 1
Joints:
- joint FL_calf_joint: limit lower=-2.818 upper=-0.888 effort=35.55 velocity=20.06 -> lower=-2.818 upper=-0.888 effort=120.0 velocity=20.06
- joint FL_hip_joint: limit lower=-0.863 upper=0.863 effort=23.7 velocity=30.1 -> lower=-0.863 upper=0.863 effort=80.0 velocity=30.1
- joint FL_thigh_joint: limit lower=-0.686 upper=4.501 effort=23.7 velocity=30.1 -> lower=-0.686 upper=4.501 effort=80.0 velocity=30.1
- joint FR_calf_joint: limit lower=-2.818 upper=-0.888 effort=35.55 velocity=20.06 -> lower=-2.818 upper=-0.888 effort=120.0 velocity=20.06
- joint FR_hip_joint: limit lower=-0.863 upper=0.863 effort=23.7 velocity=30.1 -> lower=-0.863 upper=0.863 effort=80.0 velocity=30.1
- joint FR_thigh_joint: limit lower=-0.686 upper=4.501 effort=23.7 velocity=30.1 -> lower=-0.686 upper=4.501 effort=80.0 velocity=30.1
- joint RL_calf_joint: limit lower=-2.818 upper=-0.888 effort=35.55 velocity=20.06 -> lower=-2.818 upper=-0.888 effort=120.0 velocity=20.06
- joint RL_hip_joint: limit lower=-0.863 upper=0.863 effort=23.7 velocity=30.1 -> lower=-0.863 upper=0.863 effort=80.0 velocity=30.1
- joint RL_thigh_joint: limit lower=-0.686 upper=4.501 effort=23.7 velocity=30.1 -> lower=-0.686 upper=4.501 effort=80.0 velocity=30.1
- joint RR_calf_joint: limit lower=-2.818 upper=-0.888 effort=35.55 velocity=20.06 -> lower=-2.818 upper=-0.888 effort=120.0 velocity=20.06
- joint RR_hip_joint: limit lower=-0.863 upper=0.863 effort=23.7 velocity=30.1 -> lower=-0.863 upper=0.863 effort=80.0 velocity=30.1
- joint RR_thigh_joint: limit lower=-0.686 upper=4.501 effort=23.7 velocity=30.1 -> lower=-0.686 upper=4.501 effort=80.0 velocity=30.1

File: src/quadruped_ros2_control-humble/descriptions/unitree/go1_description/xacro/const.xacro (robot description, xacro)
@@ -54,13 +54,13 @@
 	<xacro:property name="hip_position_min" value="-0.863"/>
 	<xacro:property name="hip_velocity_max" value="30.1"/>
-	<xacro:property name="hip_torque_max" value="1.0"/>
+	<xacro:property name="hip_torque_max" value="23.7"/>
 	<xacro:property name="thigh_position_max" value="4.501"/>
 	<xacro:property name="thigh_position_min" value="-2.1"/>
 	<xacro:property name="thigh_velocity_max" value="30.1"/>
-	<xacro:property name="thigh_torque_max" value="1.0"/>
+	<xacro:property name="thigh_torque_max" value="23.7"/>
 	<xacro:property name="calf_position_max" value="-0.888"/>
 	<xacro:property name="calf_position_min" value="-2.818"/>
 	<xacro:property name="calf_velocity_max" value="20.06"/>
-	<xacro:property name="calf_torque_max" value="1.0"/>
+	<xacro:property name="calf_torque_max" value="35.55"/>
 	<!-- dynamics inertial value        total 26.0382kg -->
 	<!-- trunk -->

File: src/quadruped_ros2_control-humble/descriptions/unitree/go1_description/xacro/gazebo_classic.xacro (robot description, xacro)
@@ -98,5 +98,5 @@
 		<mu1>0.6</mu1>
 		<mu2>0.6</mu2>
-		<self_collide>1</self_collide>
+		<self_collide>0</self_collide>
 		<material>Gazebo/Grey</material>
 	</gazebo>
@@ -128,13 +128,13 @@
 		<mu1>0.2</mu1>
 		<mu2>0.2</mu2>
-		<self_collide>1</self_collide>
-		<material>Gazebo/Grey</material>
-		<kp  value="1000000.0"/>
-		<kd  value="1.0"/>
+		<self_collide>0</self_collide>
+		<material>Gazebo/Grey</material>
+		<kp  value="100000.0"/>
+		<kd  value="10.0"/>
 	</gazebo>
 	<gazebo reference="FL_calf">
 		<mu1>0.2</mu1>
 		<mu2>0.2</mu2>
-		<self_collide>1</self_collide>
+		<self_collide>0</self_collide>
 		<material>Gazebo/DarkGrey</material>
 	</gazebo>
@@ -142,8 +142,8 @@
 		<mu1>0.6</mu1>
 		<mu2>0.6</mu2>
-		<self_collide>1</self_collide>
-		<material>Gazebo/DarkGrey</material>
-		<kp  value="1000000.0"/>
-		<kd  value="1.0"/>
+		<self_collide>0</self_collide>
+		<material>Gazebo/DarkGrey</material>
+		<kp  value="100000.0"/>
+		<kd  value="10.0"/>
 	</gazebo>
 	<!-- FR leg -->
@@ -156,13 +156,13 @@
 		<mu1>0.2</mu1>
 		<mu2>0.2</mu2>
-		<self_collide>1</self_collide>
-		<material>Gazebo/Grey</material>
-		<kp  value="1000000.0"/>
-		<kd  value="1.0"/>
+		<self_collide>0</self_collide>
+		<material>Gazebo/Grey</material>
+		<kp  value="100000.0"/>
+		<kd  value="10.0"/>
 	</gazebo>
 	<gazebo reference="FR_calf">
 		<mu1>0.2</mu1>
 		<mu2>0.2</mu2>
-		<self_collide>1</self_collide>
+		<self_collide>0</self_collide>
 		<material>Gazebo/DarkGrey</material>
 	</gazebo>
@@ -170,8 +170,8 @@
 		<mu1>0.6</mu1>
 		<mu2>0.6</mu2>
-		<self_collide>1</self_collide>
-		<material>Gazebo/DarkGrey</material>
-		<kp  value="1000000.0"/>
-		<kd  value="1.0"/>
+		<self_collide>0</self_collide>
+		<material>Gazebo/DarkGrey</material>
+		<kp  value="100000.0"/>
+		<kd  value="10.0"/>
 	</gazebo>
 	<!-- RL leg -->
@@ -184,13 +184,13 @@
 		<mu1>0.2</mu1>
 		<mu2>0.2</mu2>
-		<self_collide>1</self_collide>
-		<material>Gazebo/Grey</material>
-		<kp  value="1000000.0"/>
-		<kd  value="1.0"/>
+		<self_collide>0</self_collide>
+		<material>Gazebo/Grey</material>
+		<kp  value="100000.0"/>
+		<kd  value="10.0"/>
 	</gazebo>
 	<gazebo reference="RL_calf">
 		<mu1>0.2</mu1>
 		<mu2>0.2</mu2>
-		<self_collide>1</self_collide>
+		<self_collide>0</self_collide>
 		<material>Gazebo/DarkGrey</material>
 	</gazebo>
@@ -198,8 +198,8 @@
 		<mu1>0.6</mu1>
 		<mu2>0.6</mu2>
-		<self_collide>1</self_collide>
-		<material>Gazebo/DarkGrey</material>
-		<kp  value="1000000.0"/>
-		<kd  value="1.0"/>
+		<self_collide>0</self_collide>
+		<material>Gazebo/DarkGrey</material>
+		<kp  value="100000.0"/>
+		<kd  value="10.0"/>
 	</gazebo>
 	<!-- RR leg -->
@@ -212,13 +212,13 @@
 		<mu1>0.2</mu1>
 		<mu2>0.2</mu2>
-		<self_collide>1</self_collide>
-		<material>Gazebo/Grey</material>
-		<kp  value="1000000.0"/>
-		<kd  value="1.0"/>
+		<self_collide>0</self_collide>
+		<material>Gazebo/Grey</material>
+		<kp  value="100000.0"/>
+		<kd  value="10.0"/>
 	</gazebo>
 	<gazebo reference="RR_calf">
 		<mu1>0.2</mu1>
 		<mu2>0.2</mu2>
-		<self_collide>1</self_collide>
+		<self_collide>0</self_collide>
 		<material>Gazebo/DarkGrey</material>
 	</gazebo>
@@ -226,8 +226,8 @@
 		<mu1>0.6</mu1>
 		<mu2>0.6</mu2>
-		<self_collide>1</self_collide>
-		<material>Gazebo/DarkGrey</material>
-		<kp  value="1000000.0"/>
-		<kd  value="1.0"/>
+		<self_collide>0</self_collide>
+		<material>Gazebo/DarkGrey</material>
+		<kp  value="100000.0"/>
+		<kd  value="10.0"/>
 	</gazebo>
 </robot>
