Commit message: Establish stable Gazebo QP trotting baseline

File: src/quadruped_ros2_control-humble/descriptions/unitree/go1_description/xacro/gazebo_classic.xacro (robot description, xacro)
@@ -98,5 +98,5 @@
 		<mu1>0.6</mu1>
 		<mu2>0.6</mu2>
-		<self_collide>0</self_collide>
+		<self_collide>1</self_collide>
 		<material>Gazebo/Grey</material>
 	</gazebo>
@@ -128,13 +128,13 @@
 		<mu1>0.2</mu1>
 		<mu2>0.2</mu2>
-		<self_collide>0</self_collide>
-		<material>Gazebo/Grey</material>
-		<kp  value="100000.0"/>
-		<kd  value="10.0"/>
+		<self_collide>1</self_collide>
+		<material>Gazebo/Grey</material>
+		<kp  value="1000000.0"/>
+		<kd  value="1.0"/>
 	</gazebo>
 	<gazebo reference="FL_calf">
 		<mu1>0.2</mu1>
 		<mu2>0.2</mu2>
-		<self_collide>0</self_collide>
+		<self_collide>1</self_collide>
 		<material>Gazebo/DarkGrey</material>
 	</gazebo>
@@ -142,8 +142,8 @@
 		<mu1>0.6</mu1>
 		<mu2>0.6</mu2>
-		<self_collide>0</self_collide>
-		<material>Gazebo/DarkGrey</material>
-		<kp  value="100000.0"/>
-		<kd  value="10.0"/>
+		<self_collide>1</self_collide>
+		<material>Gazebo/DarkGrey</material>
+		<kp  value="1000000.0"/>
+		<kd  value="1.0"/>
 	</gazebo>
 	<!-- FR leg -->
@@ -156,13 +156,13 @@
 		<mu1>0.2</mu1>
 		<mu2>0.2</mu2>
-		<self_collide>0</self_collide>
-		<material>Gazebo/Grey</material>
-		<kp  value="100000.0"/>
-		<kd  value="10.0"/>
+		<self_collide>1</self_collide>
+		<material>Gazebo/Grey</material>
+		<kp  value="1000000.0"/>
+		<kd  value="1.0"/>
 	</gazebo>
 	<gazebo reference="FR_calf">
 		<mu1>0.2</mu1>
 		<mu2>0.2</mu2>
-		<self_collide>0</self_collide>
+		<self_collide>1</self_collide>
 		<material>Gazebo/DarkGrey</material>
 	</gazebo>
@@ -170,8 +170,8 @@
 		<mu1>0.6</mu1>
 		<mu2>0.6</mu2>
-		<self_collide>0</self_collide>
-		<material>Gazebo/DarkGrey</material>
-		<kp  value="100000.0"/>
-		<kd  value="10.0"/>
+		<self_collide>1</self_collide>
+		<material>Gazebo/DarkGrey</material>
+		<kp  value="1000000.0"/>
+		<kd  value="1.0"/>
 	</gazebo>
 	<!-- RL leg -->
@@ -184,13 +184,13 @@
 		<mu1>0.2</mu1>
 		<mu2>0.2</mu2>
-		<self_collide>0</self_collide>
-		<material>Gazebo/Grey</material>
-		<kp  value="100000.0"/>
-		<kd  value="10.0"/>
+		<self_collide>1</self_collide>
+		<material>Gazebo/Grey</material>
+		<kp  value="1000000.0"/>
+		<kd  value="1.0"/>
 	</gazebo>
 	<gazebo reference="RL_calf">
 		<mu1>0.2</mu1>
 		<mu2>0.2</mu2>
-		<self_collide>0</self_collide>
+		<self_collide>1</self_collide>
 		<material>Gazebo/DarkGrey</material>
 	</gazebo>
@@ -198,8 +198,8 @@
 		<mu1>0.6</mu1>
 		<mu2>0.6</mu2>
-		<self_collide>0</self_collide>
-		<material>Gazebo/DarkGrey</material>
-		<kp  value="100000.0"/>
-		<kd  value="10.0"/>
+		<self_collide>1</self_collide>
+		<material>Gazebo/DarkGrey</material>
+		<kp  value="1000000.0"/>
+		<kd  value="1.0"/>
 	</gazebo>
 	<!-- RR leg -->
@@ -212,13 +212,13 @@
 		<mu1>0.2</mu1>
 		<mu2>0.2</mu2>
-		<self_collide>0</self_collide>
-		<material>Gazebo/Grey</material>
-		<kp  value="100000.0"/>
-		<kd  value="10.0"/>
+		<self_collide>1</self_collide>
+		<material>Gazebo/Grey</material>
+		<kp  value="1000000.0"/>
+		<kd  value="1.0"/>
 	</gazebo>
 	<gazebo reference="RR_calf">
 		<mu1>0.2</mu1>
 		<mu2>0.2</mu2>
-		<self_collide>0</self_collide>
+		<self_collide>1</self_collide>
 		<material>Gazebo/DarkGrey</material>
 	</gazebo>
@@ -226,8 +226,8 @@
 		<mu1>0.6</mu1>
 		<mu2>0.6</mu2>
-		<self_collide>0</self_collide>
-		<material>Gazebo/DarkGrey</material>
-		<kp  value="100000.0"/>
-		<kd  value="10.0"/>
+		<self_collide>1</self_collide>
+		<material>Gazebo/DarkGrey</material>
+		<kp  value="1000000.0"/>
+		<kd  value="1.0"/>
 	</gazebo>
 </robot>
